File: Circuit/MotorDriver/MotorDriver.kicad_sch (KiCad schematic)
At the start: 28 parts, among them J3 Conn_01x03_Pin, J4 Conn_01x04_Pin, J5 Conn_01x06_Pin, J6 Conn_01x02_Pin, U3 DRV8316RRGFR, U4 XC6206PxxxMR

Commit message: コストカット
Parts:
- U4: value XC6206PxxxMR -> XC6206P332MR-G
Changed lines of the file:
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@@
 			)
 		)
-		(property "Value" "XC6206PxxxMR"
+		(property "Value" "XC6206P332MR-G"
 			(at 163.83 179.07 0)
 			(show_name no)
